File: shitpad.sch (KiCad schematic (older format))
At the start: 11 parts, among them J1 Shitty Connector, J2 Conn_01x04, J3 Conn_01x09, J4 Conn_02x05_Top_Bottom

Commit message: round 2
Parts:
- removed J4: Conn_02x05_Top_Bottom, Connector:Tag-Connect_TC2050-IDC-NL_2x05_P1.27mm_Vertical, symbol Connector_Generic:Conn_02x05_Top_Bottom
- removed JP1: VJ, Jumper:SolderJumper-2_P1.3mm_Bridged_RoundedPad1.0x1.5mm, symbol Jumper:Jumper_2_Bridged
- removed JP2: ~GJ, Jumper:SolderJumper-2_P1.3mm_Open_TrianglePad1.0x1.5mm, symbol Jumper:Jumper_2_Open
- removed JP3: GJ, Jumper:SolderJumper-2_P1.3mm_Bridged_RoundedPad1.0x1.5mm, symbol Jumper:Jumper_2_Bridged
- removed JP4: ~VJ, Jumper:SolderJumper-2_P1.3mm_Open_TrianglePad1.0x1.5mm, symbol Jumper:Jumper_2_Open
- C1: value C_Small -> 100nF
- D1: footprint LED_SMD:LED_0805_2012Metric_Pad1.15x1.40mm_HandSolder -> LED_THT:LED_D3.0mm
- R1: footprint Resistor_SMD:R_0805_2012Metric_Pad1.20x1.40mm_HandSolder -> Resistor_THT:R_Axial_DIN0207_L6.3mm_D2.5mm_P10.16mm_Horizontal
Connections:
- net +3V3: now also J1.5 (Pin_5)
- net GND: now also J1.6 (Pin_6)
- no-connect marks 3 -> 6
Other:
- moved on the sheet: C1
Changed lines of the file:
@@
 Comment4 ""
 $EndDescr
-$Comp
-L Connector_Generic:Conn_02x03_Odd_Even J1
-U 1 1 62C27F5F
-P 3550 2650
-F 0 "J1" H 3600 2967 50  0000 C CNN
-F 1 "Shitty Connector" H 3600 2876 50  0000 C CNN
-F 2 "Connector_PinSocket_2.54mm:PinSocket_2x03_P2.54mm_Vertical_SMD" H 3550 2650 50  0001 C CNN
-F 3 "~" H 3550 2650 50  0001 C CNN
-	1    3550 2650
-	1    0    0    -1
-$EndComp
-$Comp
-L power:+3V3 #PWR0101
-U 1 1 62C28C69
-P 2450 2550
-F 0 "#PWR0101" H 2450 2400 50  0001 C CNN
-F 1 "+3V3" V 2465 2678 50  0000 L CNN
-F 2 "" H 2450 2550 50  0001 C CNN
-F 3 "" H 2450 2550 50  0001 C CNN
-	1    2450 2550
-	0    -1   -1   0
-$EndComp
-$Comp
-L power:GND #PWR0102
-U 1 1 62C29354
-P 4500 2550
-F 0 "#PWR0102" H 4500 2300 50  0001 C CNN
-F 1 "GND" V 4505 2422 50  0000 R CNN
-F 2 "" H 4500 2550 50  0001 C CNN
-F 3 "" H 4500 2550 50  0001 C CNN
-	1    4500 2550
-	0    -1   -1   0
-$EndComp
-Wire Wire Line
-	4350 2550 4500 2550
-NoConn ~ 3350 2650
-NoConn ~ 3850 2650
-$Comp
-L Device:C_Small C1
-U 1 1 62C2A656
-P 2700 2250
-F 0 "C1" H 2608 2204 50  0000 R CNN
-F 1 "C_Small" H 2608 2295 50  0000 R CNN
-F 2 "Capacitor_SMD:C_0805_2012Metric_Pad1.18x1.45mm_HandSolder" H 2700 2250 50  0001 C CNN
-F 3 "~" H 2700 2250 50  0001 C CNN
-	1    2700 2250
-	-1   0    0    -1
-$EndComp
-$Comp
-L power:GND #PWR0103
-U 1 1 62C2C3C9
-P 2700 2050
-F 0 "#PWR0103" H 2700 1800 50  0001 C CNN
-F 1 "GND" H 2705 1877 50  0000 C CNN
-F 2 "" H 2700 2050 50  0001 C CNN
-F 3 "" H 2700 2050 50  0001 C CNN
-	1    2700 2050
-	-1   0    0    1
-$EndComp
-Wire Wire Line
-	2700 2150 2700 2050
 Wire Wire Line
 	5800 2700 5350 2700
@@
 $EndComp
 $Comp
-L Jumper:Jumper_2_Bridged JP1
-U 1 1 62C3E9DE
-P 3050 2550
-F 0 "JP1" H 3050 2745 50  0000 C CNN
-F 1 "VJ" H 3050 2654 50  0000 C CNN
-F 2 "Jumper:SolderJumper-2_P1.3mm_Bridged_RoundedPad1.0x1.5mm" H 3050 2550 50  0001 C CNN
-F 3 "~" H 3050 2550 50  0001 C CNN
-	1    3050 2550
-	1    0    0    -1
-$EndComp
-$Comp
-L Jumper:Jumper_2_Bridged JP3
-U 1 1 62C3F4CA
-P 4150 2550
-F 0 "JP3" H 4150 2745 50  0000 C CNN
-F 1 "GJ" H 4150 2654 50  0000 C CNN
-F 2 "Jumper:SolderJumper-2_P1.3mm_Bridged_RoundedPad1.0x1.5mm" H 4150 2550 50  0001 C CNN
-F 3 "~" H 4150 2550 50  0001 C CNN
-	1    4150 2550
-	1    0    0    -1
-$EndComp
-Wire Wire Line
-	3250 2550 3350 2550
-Wire Wire Line
-	3850 2550 3950 2550
-$Comp
-L Jumper:Jumper_2_Open JP4
-U 1 1 62C406C8
-P 4150 2950
-F 0 "JP4" H 4150 2713 50  0000 C CNN
-F 1 "~VJ" H 4150 2811 50  0000 C CNN
-F 2 "Jumper:SolderJumper-2_P1.3mm_Open_TrianglePad1.0x1.5mm" H 4150 2950 50  0001 C CNN
-F 3 "~" H 4150 2950 50  0001 C CNN
-	1    4150 2950
-	1    0    0    1
-$EndComp
-$Comp
-L Jumper:Jumper_2_Open JP2
-U 1 1 62C447D0
-P 3050 2950
-F 0 "JP2" H 3050 2713 50  0000 C CNN
-F 1 "~GJ" H 3050 2811 50  0000 C CNN
-F 2 "Jumper:SolderJumper-2_P1.3mm_Open_TrianglePad1.0x1.5mm" H 3050 2950 50  0001 C CNN
-F 3 "~" H 3050 2950 50  0001 C CNN
-	1    3050 2950
-	1    0    0    1
-$EndComp
-Wire Wire Line
-	2450 2550 2700 2550
-Wire Wire Line
-	2700 2350 2700 2550
-Connection ~ 2700 2550
-Wire Wire Line
-	2700 2550 2850 2550
-Wire Wire Line
-	3350 2750 3350 2950
-Wire Wire Line
-	3350 2950 3250 2950
-Wire Wire Line
-	3850 2750 3850 2950
-Wire Wire Line
-	3850 2950 3950 2950
-$Comp
-L power:+3V3 #PWR0108
-U 1 1 62C4AE6E
-P 4500 2950
-F 0 "#PWR0108" H 4500 2800 50  0001 C CNN
-F 1 "+3V3" V 4515 3078 50  0000 L CNN
-F 2 "" H 4500 2950 50  0001 C CNN
-F 3 "" H 4500 2950 50  0001 C CNN
-	1    4500 2950
-	0    1    1    0
-$EndComp
-$Comp
-L power:GND #PWR0109
-U 1 1 62C4BD05
-P 2450 2950
-F 0 "#PWR0109" H 2450 2700 50  0001 C CNN
-F 1 "GND" V 2455 2822 50  0000 R CNN
-F 2 "" H 2450 2950 50  0001 C CNN
-F 3 "" H 2450 2950 50  0001 C CNN
-	1    2450 2950
-	0    1    1    0
-$EndComp
-Wire Wire Line
-	2450 2950 2850 2950
-Wire Wire Line
-	4350 2950 4500 2950
-$Comp
 L Device:LED D1
 U 1 1 62C53DF0
@@
 F 0 "D1" H 2243 3767 50  0000 C CNN
 F 1 "LED" H 2243 3676 50  0000 C CNN
-F 2 "LED_SMD:LED_0805_2012Metric_Pad1.15x1.40mm_HandSolder" H 2250 3550 50  0001 C CNN
+F 2 "LED_THT:LED_D3.0mm" H 2250 3550 50  0001 C CNN
 F 3 "~" H 2250 3550 50  0001 C CNN
 	1    2250 3550
@@
 F 0 "R1" V 2443 3550 50  0000 C CNN
 F 1 "R" V 2534 3550 50  0000 C CNN
-F 2 "Resistor_SMD:R_0805_2012Metric_Pad1.20x1.40mm_HandSolder" V 2580 3550 50  0001 C CNN
+F 2 "Resistor_THT:R_Axial_DIN0207_L6.3mm_D2.5mm_P10.16mm_Horizontal" V 2580 3550 50  0001 C CNN
 F 3 "~" H 2650 3550 50  0001 C CNN
 	1    2650 3550
@@
 Text Label 5350 3000 2    50   ~ 0
 PB3
-Wire Wire Line
-	5100 4450 4650 4450
-Text Label 4650 4450 2    50   ~ 0
-SDA
-Wire Wire Line
-	5100 4850 4650 4850
-Text Label 4650 4850 2    50   ~ 0
-SCL
-Wire Wire Line
-	5100 4650 4650 4650
-Text Label 4650 4650 2    50   ~ 0
-CIPO
-Text Label 6050 4450 0    50   ~ 0
-NRST
-Wire Wire Line
-	5600 4450 6050 4450
-$Comp
-L power:+3V3 #PWR0112
-U 1 1 62C8EF21
-P 6050 4650
-F 0 "#PWR0112" H 6050 4500 50  0001 C CNN
-F 1 "+3V3" V 6065 4778 50  0000 L CNN
-F 2 "" H 6050 4650 50  0001 C CNN
-F 3 "" H 6050 4650 50  0001 C CNN
-	1    6050 4650
-	0    1    -1   0
-$EndComp
-Wire Wire Line
-	6050 4650 5600 4650
-Wire Wire Line
-	5600 4850 6050 4850
-$Comp
-L power:GND #PWR0113
-U 1 1 62C8EF15
-P 6050 4850
-F 0 "#PWR0113" H 6050 4600 50  0001 C CNN
-F 1 "GND" H 6055 4677 50  0000 C CNN
-F 2 "" H 6050 4850 50  0001 C CNN
-F 3 "" H 6050 4850 50  0001 C CNN
-	1    6050 4850
+NoConn ~ 5800 3300
+Wire Wire Line
+	5750 3500 5800 3500
+Wire Wire Line
+	3200 2750 3350 2750
+Connection ~ 3200 2750
+Wire Wire Line
+	3200 2550 3200 2750
+Wire Wire Line
+	2950 2750 3200 2750
+Wire Wire Line
+	3200 2350 3200 2250
+$Comp
+L power:GND #PWR0103
+U 1 1 62C2C3C9
+P 3200 2250
+F 0 "#PWR0103" H 3200 2000 50  0001 C CNN
+F 1 "GND" H 3205 2077 50  0000 C CNN
+F 2 "" H 3200 2250 50  0001 C CNN
+F 3 "" H 3200 2250 50  0001 C CNN
+	1    3200 2250
+	-1   0    0    1
+$EndComp
+$Comp
+L Device:C_Small C1
+U 1 1 62C2A656
+P 3200 2450
+F 0 "C1" H 3400 2350 50  0000 R CNN
+F 1 "100nF" H 3550 2550 50  0000 R CNN
+F 2 "Capacitor_SMD:C_0805_2012Metric_Pad1.18x1.45mm_HandSolder" H 3200 2450 50  0001 C CNN
+F 3 "~" H 3200 2450 50  0001 C CNN
+	1    3200 2450
 	-1   0    0    -1
 $EndComp
-$Comp
-L Connector_Generic:Conn_02x05_Top_Bottom J4
-U 1 1 62CBACDB
-P 5300 4650
-F 0 "J4" H 5350 5067 50  0000 C CNN
-F 1 "Conn_02x05_Top_Bottom" H 5350 4976 50  0000 C CNN
-F 2 "Connector:Tag-Connect_TC2050-IDC-NL_2x05_P1.27mm_Vertical" H 5300 4650 50  0001 C CNN
-F 3 "~" H 5300 4650 50  0001 C CNN
-	1    5300 4650
-	1    0    0    -1
-$EndComp
-NoConn ~ 5800 3300
-Wire Wire Line
-	5750 3500 5800 3500
+NoConn ~ 3850 2650
+NoConn ~ 3350 2650
+Wire Wire Line
+	3850 2750 4000 2750
+$Comp
+L power:GND #PWR0102
+U 1 1 62C29354
+P 4000 2750
+F 0 "#PWR0102" H 4000 2500 50  0001 C CNN
+F 1 "GND" V 4005 2622 50  0000 R CNN
+F 2 "" H 4000 2750 50  0001 C CNN
+F 3 "" H 4000 2750 50  0001 C CNN
+	1    4000 2750
+	0    -1   -1   0
+$EndComp
+$Comp
+L power:+3V3 #PWR0101
+U 1 1 62C28C69
+P 2950 2750
+F 0 "#PWR0101" H 2950 2600 50  0001 C CNN
+F 1 "+3V3" V 2965 2878 50  0000 L CNN
+F 2 "" H 2950 2750 50  0001 C CNN
+F 3 "" H 2950 2750 50  0001 C CNN
+	1    2950 2750
+	0    -1   -1   0
+$EndComp
+NoConn ~ 3850 2550
+NoConn ~ 3350 2550
+$Comp
+L Connector_Generic:Conn_02x03_Odd_Even J1
+U 1 1 62C27F5F
+P 3550 2650
+F 0 "J1" H 3600 2967 50  0000 C CNN
+F 1 "Shitty Connector" H 3600 2876 50  0000 C CNN
+F 2 "Connector_PinSocket_2.54mm:PinSocket_2x03_P2.54mm_Vertical_SMD" H 3550 2650 50  0001 C CNN
+F 3 "~" H 3550 2650 50  0001 C CNN
+	1    3550 2650
+	1    0    0    -1
+$EndComp
+NoConn ~ 4450 1850
 $EndSCHEMATC
