File: shitpad.kicad_pcb (KiCad board)
At the start: 2 copper layers, 33 x 68 mm, 20 parts, among them J1 Shitty Connector, J2 Conn_01x04, J3 Conn_01x09, J4 Conn_02x05_Top_Bottom

Commit message: round 2
Parts:
- removed the G*** at (0.00, 0.00) (x5)
- removed J4: Conn_02x05_Top_Bottom, Connector:Tag-Connect_TC2050-IDC-NL_2x05_P1.27mm_Vertical
- removed JP1: VJ, Jumper:SolderJumper-2_P1.3mm_Bridged_RoundedPad1.0x1.5mm
- removed JP2: ~GJ, Jumper:SolderJumper-2_P1.3mm_Open_TrianglePad1.0x1.5mm
- removed JP3: GJ, Jumper:SolderJumper-2_P1.3mm_Bridged_RoundedPad1.0x1.5mm
- removed JP4: ~VJ, Jumper:SolderJumper-2_P1.3mm_Open_TrianglePad1.0x1.5mm
- added G***: LOGO, shitpad:lenowo, B.Cu at (84.4, 93.2)
- added G*** (x5): LOGO, LOGO, F.Cu at (0.00, 0.00)
- C1: value C_Small -> 100nF
- D1: footprint LED_SMD:LED_0805_2012Metric_Pad1.15x1.40mm_HandSolder -> LED_THT:LED_D3.0mm
- R1: footprint Resistor_SMD:R_0805_2012Metric_Pad1.20x1.40mm_HandSolder -> Resistor_THT:R_Axial_DIN0207_L6.3mm_D2.5mm_P10.16mm_Horizontal
- moved G*** 21.7 mm to (101.4, 35.6)
- moved J1 12.2 mm to (91.0, 81.0)
- moved R1 8.31 mm to (75.4, 32.2)
- moved G*** 5.81 mm to (84.3, 67.8)
- moved J3 3.61 mm to (80.0, 48.0)
- moved D1 0.85 mm to (93.2, 31.8)
Connections:
- J1 pad 5: Net-(J1-Pad5) -> +3V3
- J1 pad 6: Net-(J1-Pad6) -> GND
Routing:
- net /CIPO: track 35.0 -> 0.00 mm, vias 2 -> 0
- net +3V3: track 121.4 -> 89.8 mm, vias 1 -> 0
- net /NRST: track 29.8 -> 0.00 mm, vias 1 -> 0
- net /SCL: track 35.1 -> 18.1 mm
- net Net-(J1-Pad6): track 15.2 -> 0.00 mm
- net /SDA: track 35.0 -> 24.3 mm, vias 2 -> 0
- net GND: track 14.4 -> 4.84 mm
- net Net-(J1-Pad5): track 9.13 -> 0.00 mm
- net Net-(J1-Pad2): track 13.5 -> 4.72 mm
- net Net-(J1-Pad4): track 0.00 -> 4.72 mm
- net Net-(J1-Pad3): track 0.00 -> 4.71 mm
- net Net-(D1-Pad2): track 6.77 -> 5.29 mm, vias 1 -> 0
- net Net-(J1-Pad1): track 6.30 -> 5.15 mm
Other:
- net class Default removed
- board text added: "I bet your bios is stock baka~"
- board text removed: "I bet your bios is stock~ baka~"
- board text removed: "in case of fuck up cut JP1 and JP3 bridge JP2 and JP4"

Commit message: ordered
Routing:
- net Net-(J1-Pad1): track 5.15 -> 12.2 mm
- net Net-(J1-Pad3): track 4.71 -> 11.7 mm
- net +3V3: track 89.8 -> 94.1 mm
- net Net-(J1-Pad2): track 4.72 -> 7.64 mm
- net Net-(J1-Pad4): track 4.72 -> 6.22 mm
- net GND: track 4.84 -> 6.00 mm
Changed lines of the file:
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@@
     (pad_to_mask_clearance 0.2)
     (pcbplotparams
-      (layerselection 0x00010f0_80000001)
+      (layerselection 0x00010f0_ffffffff)
       (disableapertmacros false)
-      (usegerberextensions false)
-      (usegerberattributes true)
-      (usegerberadvancedattributes true)
-      (creategerberjobfile true)
+      (usegerberextensions true)
+      (usegerberattributes false)
+      (usegerberadvancedattributes false)
+      (creategerberjobfile false)
       (svguseinch false)
       (svgprecision 6)
@@
       (psa4output false)
       (plotreference true)
-      (plotvalue true)
+      (plotvalue false)
       (plotinvisibletext false)
       (sketchpadsonfab false)
-      (subtractmaskfromsilk false)
+      (subtractmaskfromsilk true)
       (outputformat 1)
       (mirror false)
-      (drillshape 1)
+      (drillshape 0)
       (scaleselection 1)
       (outputdirectory "gerbers/")
@@
     (tags "LED diameter 3.0mm 2 pins")
     (attr through_hole)
-    (fp_text reference "D1" (at -2.052 0.01) (layer "B.SilkS")
+    (fp_text reference "D1" (at -2.052 0.01) (layer "B.SilkS") hide
       (effects (font (size 1 1) (thickness 0.15)) (justify mirror))
     )
-    (fp_text value "LED" (at -2.892 0) (layer "F.Fab")
+    (fp_text value "LED" (at -2.892 0) (layer "F.Fab") hide
       (effects (font (size 1 1) (thickness 0.15)))
     )
@@
     (tags "capacitor handsolder")
     (attr smd)
-    (fp_text reference "C1" (at 0 1.68) (layer "B.SilkS")
+    (fp_text reference "C1" (at 0 1.68) (layer "B.SilkS") hide
       (effects (font (size 1 1) (thickness 0.15)) (justify mirror))
     )
@@
     (fp_line (start 1 0.625) (end 1 -0.625) (layer "B.Fab") (width 0.1))
     (fp_line (start -1 -0.625) (end -1 0.625) (layer "B.Fab") (width 0.1))
-    (pad "1" smd roundrect locked (at -1.0375 0 180) (size 1.175 1.45) (layers "B.Cu" "B.Paste" "B.Mask") (roundrect_rratio 0.212766)
+    (pad "1" smd roundrect locked (at -1.0375 0 180) (size 1.175 1.45) (layers "B.Cu" "B.Paste" "B.Mask") (roundrect_rratio 0.2127659574)
       (net 1 "GND"))
-    (pad "2" smd roundrect locked (at 1.0375 0 180) (size 1.175 1.45) (layers "B.Cu" "B.Paste" "B.Mask") (roundrect_rratio 0.212766)
+    (pad "2" smd roundrect locked (at 1.0375 0 180) (size 1.175 1.45) (layers "B.Cu" "B.Paste" "B.Mask") (roundrect_rratio 0.2127659574)
       (net 2 "+3V3"))
     (model "${KISYS3DMOD}/Capacitor_SMD.3dshapes/C_0805_2012Metric.wrl"
@@
     (tags "Surface mounted socket strip SMD 2x03 2.54mm double row")
     (attr smd)
-    (fp_text reference "J1" (at 0 5.31 90) (layer "B.SilkS")
+    (fp_text reference "J1" (at 0 5.31 90) (layer "B.SilkS") hide
       (effects (font (size 1 1) (thickness 0.15)) (justify mirror))
     )
-    (fp_text value "Shitty Connector" (at 0 -5.31 90) (layer "B.Fab")
+    (fp_text value "Shitty Connector" (at 0 -5.31 90) (layer "B.Fab") hide
       (effects (font (size 1 1) (thickness 0.15)) (justify mirror))
     )
@@
     (tags "Resistor Axial_DIN0207 series Axial Horizontal pin pitch 10.16mm 0.25W = 1/4W length 6.3mm diameter 2.5mm")
     (attr through_hole)
-    (fp_text reference "R1" (at 12.332 -0.09) (layer "B.SilkS")
+    (fp_text reference "R1" (at 12.332 -0.09) (layer "B.SilkS") hide
       (effects (font (size 1 1) (thickness 0.15)) (justify mirror))
     )
@@
     (effects (font (size 1 1) (thickness 0.25)) (justify mirror))
   )
-  (gr_text "I bet your\nbios is stock\nbaka~" (at 99.314 71.882) (layer "B.SilkS")
+  (gr_text "I bet your\nbios is stock\nbaka~" (at 99.5 69.5) (layer "B.SilkS")
     (effects (font (size 1.5 1.5) (thickness 0.375)) (justify mirror))
   )
@@
   )
   (segment (start 88.46 83.52) (end 88.46 88.36) (width 1) (layer "B.Cu") (net 1))
+  (segment (start 88.46 88.36) (end 88.46 89.46) (width 1) (layer "B.Cu") (net 1))
+  (segment (start 88.46 89.46) (end 88.5 89.5) (width 1) (layer "B.Cu") (net 1))
+  (segment (start 93.51 61.99) (end 100.9125 61.99) (width 1) (layer "B.Cu") (net 2))
   (segment (start 89.23 37.202081) (end 88.882081 37.55) (width 1) (layer "B.Cu") (net 2))
   (segment (start 75.438 52.107028) (end 81.820772 58.4898) (width 1) (layer "B.Cu") (net 2))
   (segment (start 75.438 32.25) (end 75.438 52.107028) (width 1) (layer "B.Cu") (net 2))
-  (segment (start 88.46 74.4425) (end 100.9125 61.99) (width 1) (layer "B.Cu") (net 2))
   (segment (start 95.7725 56.85) (end 100.9125 61.99) (width 1) (layer "B.Cu") (net 2))
   (segment (start 89.23 36) (end 89.23 37.202081) (width 1) (layer "B.Cu") (net 2))
-  (segment (start 88.46 78.48) (end 88.46 74.4425) (width 1) (layer "B.Cu") (net 2))
+  (segment (start 88.46 67.04) (end 93.51 61.99) (width 1) (layer "B.Cu") (net 2))
   (segment (start 80.738 37.55) (end 75.438 32.25) (width 1) (layer "B.Cu") (net 2))
   (segment (start 92.83 56.85) (end 95.7725 56.85) (width 1) (layer "B.Cu") (net 2))
+  (segment (start 88.46 78.48) (end 88.46 67.04) (width 1) (layer "B.Cu") (net 2))
   (segment (start 88.882081 37.55) (end 80.738 37.55) (width 1) (layer "B.Cu") (net 2))
   (segment (start 81.820772 58.4898) (end 91.1902 58.4898) (width 1) (layer "B.Cu") (net 2))
@@
   (segment (start 91 78.48) (end 91 73.85) (width 1) (layer "B.Cu") (net 3))
   (segment (start 91 73.85) (end 91.06 73.79) (width 1) (layer "B.Cu") (net 3))
-  (segment (start 91 83.52) (end 91 88.24) (width 1) (layer "B.Cu") (net 4))
+  (segment (start 91 78.48) (end 91 71.5) (width 1) (layer "B.Cu") (net 3))
+  (segment (start 91 88) (end 91 88.24) (width 1) (layer "B.Cu") (net 4))
+  (segment (start 91 83.52) (end 91 88) (width 1) (layer "B.Cu") (net 4))
+  (segment (start 91 88) (end 91 89.5) (width 1) (layer "B.Cu") (net 4))
   (segment (start 94.31 40.04) (end 94.31 36) (width 1) (layer "B.Cu") (net 5))
   (segment (start 80 54.35) (end 94.31 40.04) (width 1) (layer "B.Cu") (net 5))
@@
   (segment (start 90.178 32.25) (end 90.678 31.75) (width 1) (layer "B.Cu") (net 7))
   (segment (start 85.598 32.25) (end 90.178 32.25) (width 1) (layer "B.Cu") (net 7))
+  (segment (start 93.54 78.48) (end 93.54 71.46) (width 1) (layer "B.Cu") (net 8))
   (segment (start 93.54 73.36) (end 93.56 73.34) (width 1) (layer "B.Cu") (net 8))
   (segment (start 93.54 78.48) (end 93.54 73.36) (width 1) (layer "B.Cu") (net 8))
+  (segment (start 93.54 86.54) (end 93.54 89.46) (width 1) (layer "B.Cu") (net 9))
+  (segment (start 93.54 83.52) (end 93.54 86.54) (width 1) (layer "B.Cu") (net 9))
   (segment (start 93.54 88.23) (end 93.53 88.24) (width 1) (layer "B.Cu") (net 9))
-  (segment (start 93.54 83.52) (end 93.54 88.23) (width 1) (layer "B.Cu") (net 9))
+  (segment (start 93.54 86.54) (end 93.54 88.23) (width 1) (layer "B.Cu") (net 9))
   (zone (net 1) (net_name "GND") (layer "B.Cu") (hatch edge 0.508)
     (connect_pads (clearance 0.508))
@@
     (polygon
       (pts
-        (xy 91.714 87.739992)
-        (xy 90.314 87.739992)
+        (xy 91.714 89.739992)
+        (xy 90.314 89.739992)
         (xy 90.314 85.189992)
         (xy 91.714 85.189992)
@@
     (polygon
       (pts
-        (xy 94.214 87.766)
-        (xy 92.814 87.766)
+        (xy 94.214 89.766)
+        (xy 92.814 89.766)
         (xy 92.814 85.216)
         (xy 94.214 85.216)
@@
         (xy 94.214 76.816)
         (xy 92.814 76.816)
-        (xy 92.814 74.266)
-        (xy 94.214 74.266)
+        (xy 92.814 71.266)
+        (xy 94.214 71.266)
       )
     )
@@
         (xy 91.714 76.816)
         (xy 90.314 76.816)
-        (xy 90.314 74.266)
-        (xy 91.714 74.266)
+        (xy 90.314 71.266)
+        (xy 91.714 71.266)
       )
     )
@@
         (xy 89.164 76.816)
         (xy 87.764 76.816)
-        (xy 87.764 74.266)
-        (xy 89.164 74.266)
+        (xy 87.764 72.766)
+        (xy 89.164 72.766)
       )
     )
@@
     (polygon
       (pts
-        (xy 89.164 87.716)
-        (xy 87.764 87.716)
+        (xy 89.164 89.716)
+        (xy 87.764 89.716)
         (xy 87.764 85.166)
         (xy 89.164 85.166)
